File: RS/RS.kicad_pcb (KiCad board)
At the start: 6 copper layers, 30 parts, among them J2 USB_C_Receptacle_USB2.0_16P, J3 Conn_02x18_Odd_Even, J4 Conn_02x18_Odd_Even, U1 NCP1117-1.5_SOT223, U2 TPD4E05U06DQA, U3 W25Q128JVS, U4 RP2040

Commit message: refresh
Parts:
- added J1: Conn_01x02_Pin, Connector_PinHeader_1.00mm:PinHeader_1x02_P1.00mm_Vertical, F.Cu at (40.4, 27.8)
- U2: moved to F.Cu
- moved R6 90.9 mm to (90.7, 105.0)
- moved R7 90.0 mm to (90.7, 106.0)
- moved U3 81.4 mm to (85.3, 116.3), turned to 180 degrees
- moved U1 72.0 mm to (83.9, 97.7)
- moved C2 68.4 mm to (86.1, 103.6), turned to 180 degrees
- moved C1 67.3 mm to (81.7, 103.6)
- moved U4 13.9 mm to (95.8, 106.7), turned to 90 degrees
- moved U2 2.08 mm to (80.8, 106.2)
Connections:
- net Net-(U4-USB_DM) renamed /USB_IN-
- net Net-(U4-USB_DP) renamed /USB_IN+
Routing:
- net VBUS: track 0.00 -> 28.6 mm
- net /QSPI_SD3: track 0.00 -> 23.5 mm
- net /QSPI_SD1: track 0.00 -> 23.3 mm
- net /QSPI_SS: track 0.00 -> 23.3 mm
- net /QSPI_SD0: track 0.00 -> 23.2 mm
- net /QSPI_SD2: track 0.00 -> 23.1 mm
- net /QSPI_SCLK: track 0.00 -> 22.9 mm
- net /USB_+: track 0.84 -> 18.0 mm, vias 1 -> 0
- net /USB_-: track 0.84 -> 17.4 mm, vias 1 -> 0
- net +3V3: track 0.00 -> 12.2 mm
- net /USB_IN-: track 0.00 -> 1.36 mm
- net /USB_IN+: track 0.00 -> 1.36 mm
- net GND: track 0.77 -> 1.48 mm, vias 0 -> 1

Commit message: refresh
Parts:
- R1, R2: footprint Resistor_SMD:R_1206_3216Metric -> Resistor_SMD:R_0402_1005Metric
- moved R4 100.0 mm to (76.2, 117.2)
- moved R5 99.0 mm to (76.2, 118.2), turned to 180 degrees
- moved J1 95.4 mm to (73.9, 117.2), turned to 180 degrees
- moved R1 62.8 mm to (83.2, 106.7), turned to 180 degrees
- moved R2 61.0 mm to (83.2, 107.7), turned to 180 degrees
- moved C12 58.8 mm to (59.5, 112.4)
- moved C13 55.8 mm to (59.5, 111.3)
Routing:
- net /QSPI_SS: track 23.3 -> 37.2 mm
- net Net-(J2-CC1): track 0.77 -> 10.0 mm, vias 0 -> 2
- net Net-(J2-CC2): track 0.77 -> 5.30 mm
- net /~{USB_BOOT}: track 0.00 -> 1.77 mm
- net +3V3: track 12.2 -> 13.1 mm, vias 0 -> 1
- net GND: track 1.48 -> 0.77 mm, vias 1 -> 0

Commit message: refresh
Parts:
- moved J3 116.6 mm to (73.9, 125.0), turned to 90 degrees
- moved J4 110.6 mm to (117.1, 86.9), turned to -90 degrees
- moved R3 110.0 mm to (112.0, 108.0)
- moved C11 86.4 mm to (112.2, 104.4)
- moved C14 86.4 mm to (115.1, 104.4)
- moved C3 86.4 mm to (114.7, 110.1)
- moved C6 86.4 mm to (109.4, 104.4)
- moved C10 86.4 mm to (105.7, 113.9)
- moved C15 86.4 mm to (115.1, 106.4)
- moved C16 86.4 mm to (115.1, 108.3)
- moved C4 86.4 mm to (114.7, 111.8)
- moved C5 86.4 mm to (114.7, 113.4)
- moved C7 86.4 mm to (109.4, 106.4)
- moved C8 86.4 mm to (105.7, 110.9)
- moved C9 86.4 mm to (109.4, 108.3)
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Other:
- board outline added: 48.1 x 41.6 mm

Commit message: refresh
Parts:
- added Y1: ABM8-272-T3, Crystal:Crystal_SMD_Abracon_ABM8G-4Pin_3.2x2.5mm, F.Cu at (104.9, 106.4)
- moved C6 62.4 mm to (170.9, 114.8)
- moved C7 62.4 mm to (170.9, 116.7)
- moved C9 62.4 mm to (170.9, 118.7)
- moved C10 62.4 mm to (167.3, 124.3)
- moved C11 62.4 mm to (173.8, 114.8)
- moved C14 62.4 mm to (176.7, 114.8)
- moved C15 62.4 mm to (176.7, 116.7)
- moved C16 62.4 mm to (176.7, 118.7)
- moved C3 62.4 mm to (176.2, 120.5)
- moved C4 62.4 mm to (176.2, 122.2)
- moved C5 62.4 mm to (176.2, 123.8)
- moved C8 62.4 mm to (167.3, 121.3)
- moved C12 51.0 mm to (163.5, 103.7)
- moved C13 51.0 mm to (163.5, 102.5)
- moved R3 10.7 mm to (101.4, 106.8), turned to 180 degrees
Routing:
- net /XIN: track 0.00 -> 4.57 mm

Commit message: refresh
Parts:
- added G***: LOGO, hi:noodles, F.Cu at (74.8, 95.2)
- moved C5 93.4 mm to (85.5, 101.8), turned to 180 degrees
- moved C10 80.2 mm to (90.7, 100.5), turned to -90 degrees
- moved C13 79.7 mm to (84.3, 111.7), turned to 180 degrees
- moved C8 79.5 mm to (89.8, 103.6)
- moved C3 73.1 mm to (104.1, 108.5)
- moved C4 72.2 mm to (106.3, 104.4)
- moved C7 70.6 mm to (101.4, 104.8)
- moved C6 70.1 mm to (101.4, 105.9)
- moved C12 62.3 mm to (101.4, 107.7), turned to 180 degrees
- moved C14 61.4 mm to (116.9, 100.9)
- moved C15 60.6 mm to (116.9, 106.5)
- moved C11 60.2 mm to (116.9, 95.2)
- moved C16 60.1 mm to (116.9, 112.1)
- moved C9 54.0 mm to (116.9, 117.8)
Connections:
- U4 pad 24: Net-(J4-Pin_31) -> Net-(J4-Pin_33)
- U4 pad 25: Net-(J4-Pin_29) -> Net-(J4-Pin_31)
- U4 pad 26: Net-(J4-Pin_33) -> Net-(J4-Pin_29)
Routing:
- net +3V3: track 13.1 -> 61.6 mm, vias 1 -> 13
- net Net-(J4-Pin_33): track 0.00 -> 32.9 mm, vias 0 -> 1
- net Net-(J4-Pin_31): track 0.00 -> 30.1 mm, vias 0 -> 1
- net Net-(J4-Pin_29): track 0.00 -> 27.8 mm, vias 0 -> 1
- net Net-(J3-Pin_4): track 0.00 -> 26.9 mm
- net Net-(J4-Pin_1): track 0.00 -> 26.7 mm
- net Net-(J3-Pin_6): track 0.00 -> 24.8 mm
- net Net-(J4-Pin_3): track 0.00 -> 24.0 mm
- net Net-(J3-Pin_8): track 0.00 -> 22.6 mm
- net Net-(J4-Pin_5): track 0.00 -> 22.5 mm
- net +1V1: track 0.00 -> 21.7 mm, vias 0 -> 2
- net Net-(J3-Pin_34): track 0.00 -> 21.2 mm
- net Net-(J4-Pin_27): track 0.00 -> 21.2 mm
- net Net-(J4-Pin_7): track 0.00 -> 21.0 mm
- net Net-(J3-Pin_10): track 0.00 -> 20.5 mm
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- added copper zone on B.Cu, net +3V3
- added copper zone on F.Cu, net GND
- added copper zone on In1.Cu, net GND
- added copper zone on In2.Cu, net GND
Other:
- copper layers 6 -> 4
- board text added: "Islam Tarek"
