File: RS/RS.kicad_pcb (KiCad board)
At the start: 4 copper layers, 48.1 x 41.6 mm, 33 parts, among them J1 Conn_01x02_Pin, J2 USB_C_Receptacle_USB2.0_16P, J3 Conn_02x18_Odd_Even, J4 Conn_02x18_Odd_Even, U1 NCP1117-1.5_SOT223, U2 TPD4E05U06DQA, U3 W25Q128JVS, U4 RP2040, Y1 ABM8-272-T3

Commit message: refresh
Parts:
- moved G*** 0.90 mm to (75.5, 95.8), turned to 90 degrees
