File: RS/RS.kicad_sch (KiCad schematic)
At the start: 32 parts, among them J1 Conn_01x02_Pin, J2 USB_C_Receptacle_USB2.0_16P, J3 Conn_02x18_Odd_Even, J4 Conn_02x18_Odd_Even, U1 NCP1117-1.5_SOT223, U2 TPD4E05U06DQA, U3 W25Q128JVS, U4 RP2040, Y1 ABM8-272-T3

Commit message: refresh
Parts:
- C1, C2: value C -> 10u; footprint (none) -> Capacitor_SMD:C_0805_2012Metric
- C10, C8: footprint (none) -> Capacitor_SMD:C_0805_2012Metric
- C11, C12, C13, C14, C15, C16, C6, C7, C9: footprint (none) -> Capacitor_SMD:C_0402_1005Metric
- C3, C4, C5: footprint (none) -> Capacitor_SMD:C_01005_0402Metric
- J3, J4: footprint (none) -> Connector_PinHeader_2.54mm:PinHeader_2x18_P2.54mm_Vertical
- R3, R4, R5, R6, R7: footprint (none) -> Resistor_SMD:R_0402_1005Metric
Connections:
- net +3V3: now also J3.2 (Pin_2)
Changed lines of the file:
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@@
 			)
 		)
-		(property "Footprint" ""
+		(property "Footprint" "Capacitor_SMD:C_0402_1005Metric"
 			(at 165.1 34.29 0)
 			(hide yes)
@@
 			)
 		)
-		(property "Footprint" ""
+		(property "Footprint" "Resistor_SMD:R_0402_1005Metric"
 			(at 161.544 75.184 90)
 			(hide yes)
@@
 			)
 		)
-		(property "Footprint" ""
+		(property "Footprint" "Capacitor_SMD:C_0402_1005Metric"
 			(at 124.46 34.29 0)
 			(hide yes)
@@
 			)
 		)
-		(property "Footprint" ""
+		(property "Footprint" "Capacitor_SMD:C_01005_0402Metric"
 			(at 86.0552 148.59 0)
 			(hide yes)
@@
 			)
 		)
-		(property "Footprint" ""
+		(property "Footprint" "Capacitor_SMD:C_0402_1005Metric"
 			(at 185.42 34.29 0)
 			(hide yes)
@@
 			)
 		)
-		(property "Footprint" ""
+		(property "Footprint" "Capacitor_SMD:C_0402_1005Metric"
 			(at 175.26 34.29 0)
 			(hide yes)
@@
 			)
 		)
-		(property "Footprint" ""
+		(property "Footprint" "Resistor_SMD:R_0402_1005Metric"
 			(at 161.544 77.724 90)
 			(hide yes)
@@
 	)
 	(symbol
+		(lib_id "power:+3V3")
+		(at 256.54 50.8 0)
+		(unit 1)
+		(body_style 1)
+		(exclude_from_sim no)
+		(in_bom yes)
+		(on_board yes)
+		(in_pos_files yes)
+		(dnp no)
+		(fields_autoplaced yes)
+		(property "Reference" "#PWR025"
+			(at 256.54 54.61 0)
+			(hide yes)
+			(show_name no)
+			(do_not_autoplace no)
+			(effects
+				(font
+					(size 1.27 1.27)
+				)
+			)
+		)
+		(property "Value" "+3V3"
+			(at 256.54 45.72 0)
+			(show_name no)
+			(do_not_autoplace no)
+			(effects
+				(font
+					(size 1.27 1.27)
+				)
+			)
+		)
+		(property "Footprint" ""
+			(at 256.54 50.8 0)
+			(hide yes)
+			(show_name no)
+			(do_not_autoplace no)
+			(effects
+				(font
+					(size 1.27 1.27)
+				)
+			)
+		)
+		(property "Datasheet" ""
+			(at 256.54 50.8 0)
+			(hide yes)
+			(show_name no)
+			(do_not_autoplace no)
+			(effects
+				(font
+					(size 1.27 1.27)
+				)
+			)
+		)
+		(property "Description" "Power symbol creates a global label with name \"+3V3\""
+			(at 256.54 50.8 0)
+			(hide yes)
+			(show_name no)
+			(do_not_autoplace no)
+			(effects
+				(font
+					(size 1.27 1.27)
+				)
+			)
+		)
+		(pin "1"
+		)
+		(instances
+			(project "RS"
+				(path "/185b82da-7a21-4bdc-a056-b46f6ab4c7d6"
+					(reference "#PWR025")
+					(unit 1)
+				)
+			)
+		)
+	)
+	(symbol
 		(lib_id "power:GND")
 		(at 256.54 93.98 0)
@@
 			)
 		)
-		(property "Footprint" ""
+		(property "Footprint" "Capacitor_SMD:C_0402_1005Metric"
 			(at 220.98 34.29 0)
 			(hide yes)
@@
 			)
 		)
-		(property "Footprint" ""
+		(property "Footprint" "Connector_PinHeader_2.54mm:PinHeader_2x18_P2.54mm_Vertical"
 			(at 264.16 71.12 0)
 			(hide yes)
@@
 			)
 		)
-		(property "Footprint" ""
+		(property "Footprint" "Capacitor_SMD:C_0805_2012Metric"
 			(at 181.3052 45.72 0)
 			(hide yes)
@@
 			)
 		)
-		(property "Footprint" ""
+		(property "Footprint" "Capacitor_SMD:C_0402_1005Metric"
 			(at 154.94 34.29 0)
 			(hide yes)
@@
 			)
 		)
-		(property "Footprint" ""
+		(property "Footprint" "Capacitor_SMD:C_01005_0402Metric"
 			(at 24.13 92.4052 0)
 			(hide yes)
@@
 			)
 		)
-		(property "Footprint" ""
+		(property "Footprint" "Capacitor_SMD:C_0402_1005Metric"
 			(at 210.82 34.29 0)
 			(hide yes)
@@
 			)
 		)
-		(property "Footprint" ""
+		(property "Footprint" "Capacitor_SMD:C_0805_2012Metric"
 			(at 216.8652 45.72 0)
 			(hide yes)
@@
 			)
 		)
-		(property "Footprint" ""
+		(property "Footprint" "Capacitor_SMD:C_0402_1005Metric"
 			(at 134.62 34.29 0)
 			(hide yes)
@@
 			)
 		)
-		(property "Value" "C"
+		(property "Value" "10u"
 			(at 97.79 35.5599 0)
 			(show_name no)
@@
 			)
 		)
-		(property "Footprint" ""
+		(property "Footprint" "Capacitor_SMD:C_0805_2012Metric"
 			(at 94.9452 38.1 0)
 			(hide yes)
@@
 			)
 		)
-		(property "Footprint" ""
+		(property "Footprint" "Connector_PinHeader_2.54mm:PinHeader_2x18_P2.54mm_Vertical"
 			(at 261.62 125.73 0)
 			(hide yes)
@@
 			)
 		)
-		(property "Footprint" ""
+		(property "Footprint" "Resistor_SMD:R_0402_1005Metric"
 			(at 47.244 112.014 90)
 			(hide yes)
@@
 			)
 		)
-		(property "Footprint" ""
+		(property "Footprint" "Capacitor_SMD:C_0402_1005Metric"
 			(at 144.78 34.29 0)
 			(hide yes)
@@
 			)
 		)
-		(property "Footprint" ""
+		(property "Footprint" "Resistor_SMD:R_0402_1005Metric"
 			(at 44.704 150.114 90)
 			(hide yes)
@@
 			)
 		)
-		(property "Footprint" ""
+		(property "Footprint" "Resistor_SMD:R_0402_1005Metric"
 			(at 49.784 144.526 90)
 			(hide yes)
@@
 			)
 		)
-		(property "Footprint" ""
+		(property "Footprint" "Capacitor_SMD:C_01005_0402Metric"
 			(at 24.13 120.3452 0)
 			(hide yes)
@@
 			)
 		)
-		(property "Value" "C"
+		(property "Value" "10u"
 			(at 72.39 35.5599 0)
 			(show_name no)
@@
 			)
 		)
-		(property "Footprint" ""
+		(property "Footprint" "Capacitor_SMD:C_0805_2012Metric"
 			(at 69.5452 38.1 0)
 			(hide yes)

Commit message: refresh
Parts:
- J1: footprint (none) -> Connector_PinHeader_1.00mm:PinHeader_1x02_P1.00mm_Vertical
Connections:
- net USB_IN-: now reaches R6.2, U4.46 (USB_DM)
- net USB_IN+: now reaches R7.2, U4.47 (USB_DP)
Other:
- moved on the sheet: R6, R7
Changed lines of the file:
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@@
 	(wire
 		(pts
+			(xy 157.48 76.2) (xy 165.1 76.2)
+		)
+		(stroke
+			(width 0)
+			(type default)
+		)
+	)
+	(wire
+		(pts
 			(xy 45.72 43.18) (xy 48.26 45.72)
 		)
@@
 	(wire
 		(pts
-			(xy 144.78 78.74) (xy 157.48 78.74)
+			(xy 144.78 78.74) (xy 149.86 78.74)
 		)
 		(stroke
@@
 	(wire
 		(pts
+			(xy 157.48 78.74) (xy 165.1 78.74)
+		)
+		(stroke
+			(width 0)
+			(type default)
+		)
+	)
+	(wire
+		(pts
 			(xy 269.24 146.05) (xy 269.24 148.59)
 		)
@@
 	(wire
 		(pts
-			(xy 144.78 76.2) (xy 157.48 76.2)
+			(xy 144.78 76.2) (xy 149.86 76.2)
 		)
 		(stroke
@@
 		)
 	)
+	(label "USB_IN-"
+		(at 157.48 76.2 0)
+		(effects
+			(font
+				(size 1.27 1.27)
+			)
+			(justify left bottom)
+		)
+	)
 	(label "QSPI_SD3"
 		(at 50.8 163.83 0)
@@
 		)
 	)
+	(label "USB_IN+"
+		(at 157.48 78.74 0)
+		(effects
+			(font
+				(size 1.27 1.27)
+			)
+			(justify left bottom)
+		)
+	)
 	(symbol
 		(lib_id "Device:C_Small")
@@
 	(symbol
 		(lib_id "Device:R_US")
-		(at 161.29 76.2 90)
+		(at 153.67 76.2 90)
 		(unit 1)
 		(body_style 1)
@@
 		(dnp no)
 		(property "Reference" "R6"
-			(at 161.29 71.12 90)
+			(at 153.67 71.12 90)
 			(show_name no)
 			(do_not_autoplace no)
@@
 		)
 		(property "Value" "27"
-			(at 161.29 73.66 90)
+			(at 153.67 73.66 90)
 			(show_name no)
 			(do_not_autoplace no)
@@
 		)
 		(property "Footprint" "Resistor_SMD:R_0402_1005Metric"
-			(at 161.544 75.184 90)
+			(at 153.924 75.184 90)
 			(hide yes)
 			(show_name no)
@@
 		)
 		(property "Datasheet" ""
-			(at 161.29 76.2 0)
+			(at 153.67 76.2 0)
 			(hide yes)
 			(show_name no)
@@
 		)
 		(property "Description" "Resistor, US symbol"
-			(at 161.29 76.2 0)
+			(at 153.67 76.2 0)
 			(hide yes)
 			(show_name no)
@@
 	(symbol
 		(lib_id "Device:R_US")
-		(at 161.29 78.74 90)
+		(at 153.67 78.74 90)
 		(unit 1)
 		(body_style 1)
@@
 		(dnp no)
 		(property "Reference" "R7"
-			(at 161.29 81.534 90)
+			(at 153.67 81.534 90)
 			(show_name no)
 			(do_not_autoplace no)
@@
 		)
 		(property "Value" "27"
-			(at 161.29 83.82 90)
+			(at 153.67 83.82 90)
 			(show_name no)
 			(do_not_autoplace no)
@@
 		)
 		(property "Footprint" "Resistor_SMD:R_0402_1005Metric"
-			(at 161.544 77.724 90)
+			(at 153.924 77.724 90)
 			(hide yes)
 			(show_name no)
@@
 		)
 		(property "Datasheet" ""
-			(at 161.29 78.74 0)
+			(at 153.67 78.74 0)
 			(hide yes)
 			(show_name no)
@@
 		)
 		(property "Description" "Resistor, US symbol"
-			(at 161.29 78.74 0)
+			(at 153.67 78.74 0)
 			(hide yes)
 			(show_name no)
@@
 			)
 		)
-		(property "Footprint" ""
+		(property "Footprint" "Connector_PinHeader_1.00mm:PinHeader_1x02_P1.00mm_Vertical"
 			(at 21.59 151.13 0)
 			(hide yes)

Commit message: refresh
Parts:
- R1, R2: footprint Resistor_SMD:R_1206_3216Metric -> Resistor_SMD:R_0402_1005Metric
Changed lines of the file:
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@@
 			)
 		)
-		(property "Footprint" "Resistor_SMD:R_1206_3216Metric"
+		(property "Footprint" "Resistor_SMD:R_0402_1005Metric"
 			(at 58.166 34.544 90)
 			(hide yes)
@@
 			)
 		)
-		(property "Footprint" "Resistor_SMD:R_1206_3216Metric"
+		(property "Footprint" "Resistor_SMD:R_0402_1005Metric"
 			(at 58.166 37.084 90)
 			(hide yes)

Commit message: refresh
Parts:
- Y1: footprint ABM8-272-T3:XTAL_ABM8-272-T3 -> Crystal:Crystal_SMD_Abracon_ABM8G-4Pin_3.2x2.5mm
Changed lines of the file:
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@@
 			)
 		)
-		(property "Footprint" "ABM8-272-T3:XTAL_ABM8-272-T3"
+		(property "Footprint" "Crystal:Crystal_SMD_Abracon_ABM8G-4Pin_3.2x2.5mm"
 			(at 31.75 105.41 0)
 			(hide yes)

Commit message: refresh
Connections:
- net at U4.24 (SWCLK): now also J4.33 (Pin_33); no longer J4.31 (Pin_31)
- net at U4.25 (SWDIO): now also J4.31 (Pin_31); no longer J4.29 (Pin_29)
- net at U4.26 (RUN): now also J4.29 (Pin_29); no longer J4.33 (Pin_33)
Changed lines of the file:
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@@
-	(wire
-		(pts
-			(xy 160.02 124.46) (xy 160.02 143.51)
-		)
-		(stroke
-			(width 0)
-			(type default)
-		)
-	)
 	(wire
 		(pts
@@
 	(wire
 		(pts
+			(xy 162.56 143.51) (xy 256.54 143.51)
+		)
+		(stroke
+			(width 0)
+			(type default)
+		)
+	)
+	(wire
+		(pts
 			(xy 269.24 58.42) (xy 269.24 60.96)
 		)
@@
 	(wire
 		(pts
-			(xy 162.56 127) (xy 162.56 140.97)
+			(xy 162.56 127) (xy 162.56 143.51)
 		)
 		(stroke
@@
 	(wire
 		(pts
+			(xy 160.02 124.46) (xy 160.02 146.05)
+		)
+		(stroke
+			(width 0)
+			(type default)
+		)
+	)
+	(wire
+		(pts
 			(xy 220.98 135.89) (xy 256.54 135.89)
 		)
@@
 	(wire
 		(pts
-			(xy 142.24 146.05) (xy 256.54 146.05)
-		)
-		(stroke
-			(width 0)
-			(type default)
-		)
-	)
-	(wire
-		(pts
 			(xy 44.45 48.26) (xy 48.26 48.26)
 		)
@@
 	(wire
 		(pts
-			(xy 162.56 140.97) (xy 256.54 140.97)
-		)
-		(stroke
-			(width 0)
-			(type default)
-		)
-	)
-	(wire
-		(pts
 			(xy 269.24 81.28) (xy 269.24 83.82)
 		)
@@
 	(wire
 		(pts
-			(xy 160.02 143.51) (xy 256.54 143.51)
-		)
-		(stroke
-			(width 0)
-			(type default)
-		)
-	)
-	(wire
-		(pts
 			(xy 215.9 60.96) (xy 256.54 60.96)
 		)
@@
 	(wire
 		(pts
+			(xy 256.54 140.97) (xy 142.24 140.97)
+		)
+		(stroke
+			(width 0)
+			(type default)
+		)
+	)
+	(wire
+		(pts
 			(xy 220.98 127) (xy 220.98 135.89)
 		)
@@
 	(wire
 		(pts
-			(xy 142.24 68.58) (xy 142.24 146.05)
-		)
-		(stroke
-			(width 0)
-			(type default)
-		)
-	)
-	(wire
-		(pts
 			(xy 44.45 30.48) (xy 48.26 30.48)
 		)
@@
 	(wire
 		(pts
+			(xy 256.54 146.05) (xy 160.02 146.05)
+		)
+		(stroke
+			(width 0)
+			(type default)
+		)
+	)
+	(wire
+		(pts
 			(xy 223.52 124.46) (xy 223.52 133.35)
 		)
@@
 		)
 		(stroke
+			(width 0)
+			(type default)
+		)
+	)
+	(wire
+		(pts
+			(xy 142.24 68.58) (xy 142.24 140.97)
+		)
+		(stroke
